File: schematic_kicad/shortwave.sch (KiCad schematic (older format))
At the start: 45 parts, among them J1 AudioJack2, Q1 2N3904, Q2 2N3904, U1 74HC4051, U2 74HCT4046, U3 NE5532

Commit message: updated schematic
Parts:
- added C16: 100u, symbol Device:CP
Connections:
- net +5V: now also C16.1
- net GND: now also C16.2
Other:
- note added: "a 74xx based shortwave receiver\n2021 by Michael Wiebusch"
- note added: "all the info and details about the project\nhttps://acidbourbon.wordpress.com/2021/04/11/a-74xx-defined-radio/"
Changed lines of the file:
@@
 Wire Wire Line
 	8400 2850 9600 2850
+Text Notes 8900 9550 0    118  ~ 0
+all the info and details about the project\nhttps://acidbourbon.wordpress.com/2021/04/11/a-74xx-defined-radio/
+Text Notes 8900 7600 0    157  ~ 0
+a 74xx based shortwave receiver\n2021 by Michael Wiebusch
+$Comp
+L Device:CP C16
+U 1 1 6074F91B
+P 3350 6950
+F 0 "C16" H 3468 6996 50  0000 L CNN
+F 1 "100u" H 3468 6905 50  0000 L CNN
+F 2 "" H 3388 6800 50  0001 C CNN
+F 3 "~" H 3350 6950 50  0001 C CNN
+	1    3350 6950
+	1    0    0    -1
+$EndComp
+Wire Wire Line
+	3800 6700 3350 6700
+Wire Wire Line
+	3350 6700 3350 6800
+Wire Wire Line
+	3350 7100 3350 7200
+$Comp
+L power:GND #PWR031
+U 1 1 6075822F
+P 3350 7200
+F 0 "#PWR031" H 3350 6950 50  0001 C CNN
+F 1 "GND" H 3355 7027 50  0000 C CNN
+F 2 "" H 3350 7200 50  0001 C CNN
+F 3 "" H 3350 7200 50  0001 C CNN
+	1    3350 7200
+	1    0    0    -1
+$EndComp
 $EndSCHEMATC

Commit message: cosmetics
Other:
- note added: "Volume Pot"
Changed lines of the file:
@@
 	1    0    0    -1
 $EndComp
+Text Notes 13950 3550 0    118  ~ 0
+Volume Pot
 $EndSCHEMATC

Commit message: more cosmetics
Other:
- note added: "Volume\nPot"
- note added: "active half wave\nrectifier"
- note removed: "Volume Pot"
Changed lines of the file:
@@
 Wire Wire Line
 	8400 2850 9600 2850
-Text Notes 8900 9550 0    118  ~ 0
+Text Notes 8700 9450 0    118  ~ 0
 all the info and details about the project\nhttps://acidbourbon.wordpress.com/2021/04/11/a-74xx-defined-radio/
-Text Notes 8900 7600 0    157  ~ 0
+Text Notes 8700 8200 0    157  ~ 0
 a 74xx based shortwave receiver\n2021 by Michael Wiebusch
 $Comp
@@
 	1    0    0    -1
 $EndComp
-Text Notes 13950 3550 0    118  ~ 0
-Volume Pot
+Text Notes 14000 3750 0    118  ~ 0
+Volume\nPot
+Text Notes 11150 4700 0    118  ~ 0
+active half wave\nrectifier
 $EndSCHEMATC
